File: ecad/kicad/wall-sensor-advanced/ukmarsbot-wall-sensor-advanced.kicad_pcb (KiCad board)
At the start: 2 copper layers, 27.3 x 80 mm, 31 parts, among them J1 Conn_01x14, Q1 TEFT4300, Q2 TEFT4300, Q3 TEFT4300, Q4 TEFT4300, Q5 BC337, Q6 BC337

Commit message: Zwischenstand: IBOM, Layout
Parts:
- added FID1: Fiducial_0.75mm_Mask1.5mm, Fiducial:Fiducial_0.75mm_Mask1.5mm, F.Cu at (141.5, 143.5)
- added FID2: Fiducial_0.75mm_Mask1.5mm, Fiducial:Fiducial_0.75mm_Mask1.5mm, F.Cu at (140.0, 68.5)
- added FID3: Fiducial_0.75mm_Mask1.5mm, Fiducial:Fiducial_0.75mm_Mask1.5mm, F.Cu at (155.0, 67.5)
