File: ecad/kicad/mainboard/mainboard.kicad_pcb (KiCad board)
At the start: 2 copper layers, 99.1 x 81.3 mm, 37 parts, among them IC1 74HC86, J1 SENSORS, J2 CONN_06SILK_FEMALE_PTH, J3 CONN_06SILK_FEMALE_PTH, J4 POWER, J5 SERIAL, M1 Left Motor, M2 Right Motor, U1 Arduino_Nano, U2 TB6612FNG-Module

Commit message: layout
Routing:
- net 5V: track 220.0 -> 237.5 mm
- net /USER_IO: track 54.3 -> 37.4 mm, vias 2 -> 0
- net /LEFT_PWM: track 29.6 -> 32.9 mm
- net /RIGHT_A: track 47.3 -> 44.5 mm
- net //LEFT_DIR: track 22.8 -> 24.8 mm, vias 2 -> 1
- net /RIGHT_B: track 46.4 -> 44.4 mm
- net unconnected-(S1-Pad1): track 0.00 -> 1.50 mm
- net /LEFT_MOTOR_2: track 47.9 -> 46.8 mm
- net /RIGHT_CLK_A: track 12.7 -> 13.6 mm
- net /EMITTER_A: track 23.1 -> 23.6 mm
- net /V_BATT: track 86.7 -> 86.2 mm
- net //RIGHT_DIR: track 43.4 -> 43.1 mm, vias 3 -> 1
- net /BATTERY_VOLTS: track 18.8 -> 18.7 mm, vias 2 -> 0
- net /FUNCTION_SELECT: vias 2 -> 1

Commit message: Layout fertig (fast)
Parts:
- C2, C3: footprint Capacitor_THT:CP_Radial_D8.0mm_P2.50mm -> Capacitor_THT:CP_Radial_D10.0mm_P5.00mm
- moved C3 1.80 mm to (137.7, 141.4)
Routing:
- net GND: track 118.0 -> 244.2 mm, vias 3 -> 8
- net Net-(S3A-2): track 42.7 -> 49.5 mm, vias 0 -> 1
- net /FUNCTION_SELECT: track 122.8 -> 128.4 mm, vias 1 -> 2
- net /RIGHT_PWM: track 44.4 -> 49.8 mm, vias 1 -> 2
- net /LEFT_CLK_A: track 4.60 -> 9.64 mm
- net /LEFT_A: track 50.4 -> 53.9 mm, vias 1 -> 2
- net /LEFT_PWM: track 32.9 -> 29.6 mm, vias 2 -> 0
- net /RIGHT_DIR: track 73.3 -> 76.3 mm, vias 2 -> 3
- net /LEFT_MOTOR_1: track 47.7 -> 44.7 mm
- net Net-(S3C-2): track 56.3 -> 59.0 mm
- net /LEFT_MOTOR_2: track 46.8 -> 44.5 mm
- net /RXD_BT: track 34.9 -> 33.0 mm
- net /LEFT_DIR: track 46.2 -> 44.5 mm, vias 1 -> 3
- net 5V: track 237.5 -> 235.9 mm, vias 0 -> 2
- net unconnected-(S1-O-Pad1): track 1.50 -> 0.00 mm
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- added copper zone on F.Cu, net GND
Other:
- outline, holes or cut-outs redrawn

Commit message: final layout 1.3cw
Parts:
- C2, C3: value 330uF, 16V -> 220uF, 16V; footprint Capacitor_THT:CP_Radial_D10.0mm_P5.00mm -> Capacitor_SMD:CP_Elec_8x10
- S1: footprint ukmarsbot:SW_MINI-SPDT-RTECH-78-0564 -> ukmarsbot:SW_MINI-SPDT-SW
- moved C3 3.23 mm to (134.6, 140.5), turned to -90 degrees
- moved C2 1.45 mm to (125.8, 140.5), turned to -90 degrees
Connections:
- S1 pad 1: unconnected-(S1-O-Pad1) -> (no net)
Routing:
- net /V_BATT: track 87.1 -> 83.0 mm, vias 1 -> 0
- net /RIGHT_PWM: track 49.8 -> 53.4 mm
- net GND: track 244.2 -> 242.3 mm, vias 8 -> 9
- net 5V: track 235.9 -> 234.1 mm, vias 2 -> 3
- net /RIGHT_DIR: track 76.3 -> 77.8 mm
- net (no net): track 1.50 -> 0.00 mm
- net //RIGHT_DIR: track 43.3 -> 41.8 mm
Other:
- board text added: "V1.3cw"
