File: ecad/kicad/mainboard/mainboard.kicad_sch (KiCad schematic)
At the start: 34 parts, among them IC1 74HC86, J1 SENSORS, J2 CONN_06SILK_FEMALE_PTH, J3 CONN_06SILK_FEMALE_PTH, J4 POWER, J5 SERIAL, M1 Left Motor, M2 Right Motor, U1 Arduino_Nano, U2 TB6612FNG-Module

Commit message: Layout fertig (fast)
Parts:
- C2, C3: footprint Capacitor_THT:CP_Radial_D8.0mm_P2.50mm -> Capacitor_THT:CP_Radial_D10.0mm_P5.00mm
Changed lines of the file:
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@@
 			)
 		)
-		(property "Footprint" "Capacitor_THT:CP_Radial_D8.0mm_P2.50mm"
+		(property "Footprint" "Capacitor_THT:CP_Radial_D10.0mm_P5.00mm"
 			(at 97.4852 85.09 0)
 			(effects
@@
 			)
 		)
-		(property "Footprint" "Capacitor_THT:CP_Radial_D8.0mm_P2.50mm"
+		(property "Footprint" "Capacitor_THT:CP_Radial_D10.0mm_P5.00mm"
 			(at 78.4352 85.09 0)
 			(effects

Commit message: final layout 1.3cw
Parts:
- C2, C3: value 330uF, 16V -> 220uF, 16V; footprint Capacitor_THT:CP_Radial_D10.0mm_P5.00mm -> Capacitor_SMD:CP_Elec_8x10
- S1: footprint ukmarsbot:SW_MINI-SPDT-RTECH-78-0564 -> ukmarsbot:SW_MINI-SPDT-SW
Changed lines of the file:
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@@
 			)
 		)
-		(property "Value" "330uF, 16V"
+		(property "Value" "220uF, 16V"
 			(at 97.155 83.82 0)
 			(effects
@@
 			)
 		)
-		(property "Footprint" "Capacitor_THT:CP_Radial_D10.0mm_P5.00mm"
+		(property "Footprint" "Capacitor_SMD:CP_Elec_8x10"
 			(at 97.4852 85.09 0)
 			(effects
@@
 			)
 		)
-		(property "Value" "330uF, 16V"
+		(property "Value" "220uF, 16V"
 			(at 80.391 82.0932 0)
 			(effects
@@
 			)
 		)
-		(property "Footprint" "Capacitor_THT:CP_Radial_D10.0mm_P5.00mm"
+		(property "Footprint" "Capacitor_SMD:CP_Elec_8x10"
 			(at 78.4352 85.09 0)
 			(effects
@@
 			)
 		)
-		(property "Footprint" "ukmarsbot:SW_MINI-SPDT-RTECH-78-0564"
+		(property "Footprint" "ukmarsbot:SW_MINI-SPDT-SW"
 			(at 227.33 34.29 0)
 			(effects
